Commit message: removed comments

File: urdf/gazebo.xacro (robot description, xacro)
@@ -17,13 +17,4 @@
     <material>Gazebo/Blue</material>
   </gazebo>
-  <!-- <gazebo reference="kinect_sensor_link">
-    <material>Gazebo/Red</material>
-  </gazebo>
-   <gazebo reference="imu_sensor_link">
-    <material>Gazebo/Yellow</material>
-  </gazebo>
-  <gazebo reference="camera_link">
-    <material>Gazebo/Blue</material>
-  </gazebo>  -->
   <gazebo>
     <plugin filename="libgazebo_ros_diff_drive.so" name="differential_drive_controller">

File: urdf/rc_car.xacro (robot description, xacro)
@@ -8,12 +8,4 @@
   <xacro:joint_wheel name="joint_left_wheel" child_link="link_left_wheel" origin_xyz="-0.05 -0.15 0" />
   <xacro:joint_wheel name="joint_right_wheel" child_link="link_right_wheel" origin_xyz="-0.05 0.15 0" />
-  <!-- <link name="base_link"/>
-  <joint name="base" type="fixed">
-    <origin xyz="0.0 0.0 0.0" rpy="0.0 0.0 0.0"/>
-    <parent link="base_link"/>
-    <child link="link_chassis"/>
-    <axis xyz="0.0 0.0 0.0"/>
-    <limit lower="0.0" upper="0.0" effort="0.0" velocity="0.0"/>
-  </joint> -->
   <link name="link_chassis">
     <!-- pose and inertial -->
@@ -60,110 +52,3 @@
     </visual>
     </link>
-    <!-- laser scanner sensor -->
-   <!-- <link name="sensor_laser">
-    <inertial>
-      <origin xyz="0 0 0" rpy="0 0 0" />
-      <mass value="0.01" />
-      <xacro:cylinder_inertia mass="1" r="0.05" l="0.1" />
-   </inertial>
-    <visual>
-      <origin xyz="0 0 0" rpy="0 0 0" />
-      <geometry>
-        <cylinder radius="0.025" length="0.1"/>
-      </geometry>
-      <material name="white" />
-    </visual>
-    <collision>
-      <origin xyz="0 0 0" rpy="0 0 0"/>
-      <geometry>
-        <cylinder radius="0.025" length="0.1"/>
-      </geometry>
-    </collision>
-  </link>
-  <joint name="joint_sensor_laser" type="fixed">
-    <origin xyz="0.05 0 0.05" rpy="0 0 0"/>
-    <parent link="link_chassis"/>
-    <child link="sensor_laser"/>
-  </joint>
-  <! imu sensor -->
-    <!-- <link name="imu_sensor_link">
-    <inertial>
-      <origin xyz="0 0 0" rpy="0 0 0" />
-      <mass value="1" />
-      <xacro:cylinder_inertia mass="1" r="0.0025" l="0.025" />
-   </inertial>
-    <visual>
-      <origin xyz="0 0 0" rpy="0 0 0" />
-      <geometry>
-        <cylinder radius="0.025" length="0.05"/>
-      </geometry>
-      <material name="white" />
-    </visual>
-    <collision>
-      <origin xyz="0 0 0" rpy="0 0 0"/>
-      <geometry>
-        <cylinder radius="0.05" length="0.1"/>
-      </geometry>
-    </collision>
-  </link>
-  <joint name="imu_joint" type="fixed">
-    <origin xyz="-0.20 0.00 0.05" rpy="0 0 0"/>
-    <parent link="link_chassis"/>
-    <child link="imu_sensor_link"/>
-  </joint>
-  <! kinect -->
-     <!-- <link name="kinect_sensor_link">
-    <inertial>
-      <origin xyz="0 0 0" rpy="0 0 1.57" />
-      <mass value="0.01" />
-      <xacro:cylinder_inertia mass="0.01" r="0.0025" l="0.025" />
-   </inertial>
-    <visual>
-      <origin xyz="0 0 0" rpy="0 0 1.58" />
-      <geometry>
-          <mesh filename="package://robotnik_sensors/meshes/kinect.dae"/>
-        <cylinder radius="0.025" length="0.05"/>
-      </geometry>
-      <material name="white" />
-    </visual>
-    <collision>
-      <origin xyz="0 0 0" rpy="0 0 0"/>
-      <geometry>
-        <cylinder radius="0.025" length="0.1"/>
-      </geometry>
-    </collision>
-  </link>
-  <joint name="kinect_joint" type="fixed">
-    <origin xyz="0.10 0.00 0.05" rpy="0 0 0"/>
-    <parent link="link_chassis"/>
-    <child link="kinect_sensor_link"/>
-  </joint>
-     <link name="camera_link">
-    <inertial>
-      <origin xyz="0 0 0" rpy="0 0 0" />
-      <mass value="0.01" />
-      <xacro:cylinder_inertia mass="0.01" r="0.0025" l="0.025" />
-   </inertial>
-    <visual>
-      <origin xyz="0 0 0" rpy="0 0 1.57" />
-      <geometry>
-           <! <mesh filename="package://robotnik_sensors/meshes/camera_axis_p5514.dae"/> --> -->
-                   <!-- <cylinder radius="0.025" length="0.05"/>
-        <cylinder radius="0.025" length="0.05"/>
-        <cylinder radius="0.025" length="0.05"/>
-      </geometry>
-      <material name="white" />
-    </visual>
-    <collision>
-      <origin xyz="0 0 0" rpy="0 0 0"/>
-      <geometry>
-        <cylinder radius="0.025" length="0.1"/>
-      </geometry>
-    </collision>
-  </link>
-  <joint name="camera_joint" type="fixed">
-    <origin xyz="0.20 0.00 0.05" rpy="0 0 0"/>
-    <parent link="link_chassis"/>
-    <child link="camera_link"/>
-  </joint>    -->
   </robot>
